File: kicad/panstamp-nrg/panstamp.sch (KiCad schematic (older format))
At the start: 55 parts, among them P1 CONN_12, P2 CONN_12, P3 CONN_5, U1 CC430F5137, U3 SI7021, U4 MMA8652FC, X1 26MHz

Commit message: Final 1.0 version
Connections:
- net P1.2: no longer U4.5 (INT2)
- net P1.3: no longer U4.3 (INT1)
- net P3.3: no longer U4.1 (VDD)
- net P3.6: now also U4.5 (INT2)
- net P3.7: now also U4.1 (VDD)
- no-connect marks 0 -> 1
Changed lines of the file:
@@
 	3850 9300 3400 9300
-Wire Wire Line
-	3850 9550 3400 9550
 Wire Wire Line
 	3850 9700 3400 9700
@@
 Text Label 14300 8000 2    60   ~ 0
 I2C_SCL
-Text Label 3400 9550 0    60   ~ 0
-P1.3
 Text Label 3400 9700 0    60   ~ 0
-P1.2
+P3.6
 $Comp
 L VCC #PWR034
@@
 	0    -1   -1   0
 $EndComp
-Text Notes 7600 8100 0    60   ~ 0
-CL=((C1 x C2) / (C1 + C2)) + 2.5p
 Text Label 3400 8650 0    60   ~ 0
-P3.3
+P3.7
 $Comp
 L VCC #PWR039
@@
 Text Label 2700 9650 2    60   ~ 0
 P2.1/A1
+NoConn ~ 3850 9550
+Text Notes 7600 8100 0    60   ~ 0
+CL=((C1 x C2) / (C1 + C2)) + 2.5p
 $EndSCHEMATC

Commit message: New 1.1 version released
Parts:
- removed C30: 10u, SM0603S, symbol C
- R1: footprint SM0603 -> SM0402
- TH1: footprint SM0603S -> SM0402
Connections:
- net I2C_SCL: now also U1.4 (P1.7/(PM)); no longer U1.6 (P1.5/(PM))
- net P1.3: now also U4.5 (INT2)
- net P2.1/A1: no longer R1.1, TH1.1
- net P2.2/A2: no longer TH1.2
- net P2.5/A5: now also R1.1, TH1.1
- net P3.6: now also TH1.2; no longer U4.5 (INT2)
- net P1.7 renamed P1.5
- net P1.5: now also U1.6 (P1.5/(PM)); no longer U1.4 (P1.7/(PM))
Changed lines of the file:
@@
 EESchema Schematic File Version 2
 LIBS:power
-LIBS:device
-LIBS:transistors
-LIBS:conn
-LIBS:linear
-LIBS:regul
-LIBS:74xx
-LIBS:cmos4000
-LIBS:adc-dac
-LIBS:memory
-LIBS:xilinx
-LIBS:special
-LIBS:microcontrollers
-LIBS:dsp
-LIBS:microchip
-LIBS:analog_switches
-LIBS:motorola
-LIBS:texas
-LIBS:intel
-LIBS:audio
-LIBS:interface
-LIBS:digital-audio
-LIBS:philips
-LIBS:display
-LIBS:cypress
-LIBS:siliconi
-LIBS:opto
-LIBS:atmel
-LIBS:contrib
-LIBS:valves
-LIBS:atmega8
-LIBS:atmel89cxxxx
-LIBS:atmel-1
-LIBS:atmel-2005
-LIBS:avr
-LIBS:avr-1
-LIBS:avr-2
-LIBS:avr-3
-LIBS:avr-4
-LIBS:hopf
-LIBS:rfm-ash
-LIBS:mycomponents
 LIBS:panstamp-cache
 EELAYER 24 0
@@
 Text Label 12250 7900 0    60   ~ 0
 P1.4
-Text Label 12250 8000 0    60   ~ 0
+Text Label 12250 8200 0    60   ~ 0
 P1.5
 Text Label 12250 8100 0    60   ~ 0
 P1.6
-Text Label 12250 8200 0    60   ~ 0
+Text Label 12250 8000 0    60   ~ 0
 P1.7
 Text Label 11300 8500 0    60   ~ 0
@@
 F 0 "TH1" V 2400 9350 50  0000 C CNN
 F 1 "THERMISTOR" V 2200 9300 50  0000 C CNN
-F 2 "SM0603S" H 2300 9300 60  0001 C CNN
+F 2 "SM0402" H 2300 9300 60  0001 C CNN
 F 3 "" H 2300 9300 60  0000 C CNN
 	1    2300 9300
@@
 F 0 "R1" V 2380 10000 40  0000 C CNN
 F 1 "10k" V 2307 10001 40  0000 C CNN
-F 2 "SM0603" V 2230 10000 30  0001 C CNN
+F 2 "SM0402" V 2230 10000 30  0001 C CNN
 F 3 "" H 2300 10000 30  0001 C CNN
 	1    2300 10000
@@
 P1.6
 Text Label 13650 6100 0    60   ~ 0
-P1.7
+P1.5
 $Comp
 L C C6
@@
 	13450 8200 14300 8200
 Text Label 13450 8200 0    60   ~ 0
-P1.7
+P1.5
 Text Label 13450 8100 0    60   ~ 0
 P1.6
 Text Label 13450 8000 0    60   ~ 0
-P1.5
+P1.7
 Text Label 13450 7900 0    60   ~ 0
 P1.4
@@
 I2C_SCL
 Text Label 3400 9700 0    60   ~ 0
-P3.6
+P1.3
 $Comp
 L VCC #PWR034
@@
 	-1   0    0    1
 $EndComp
-$Comp
-L C C30
-U 1 1 533568D9
-P 4350 6150
-F 0 "C30" H 4400 6250 50  0000 L CNN
-F 1 "10u" H 4400 6050 50  0000 L CNN
-F 2 "SM0603S" H 4350 6150 60  0001 C CNN
-F 3 "" H 4350 6150 60  0001 C CNN
-	1    4350 6150
-	1    0    0    -1
-$EndComp
-$Comp
-L GND #PWR043
-U 1 1 533568EC
-P 4350 6450
-F 0 "#PWR043" H 4350 6450 30  0001 C CNN
-F 1 "GND" H 4350 6380 30  0001 C CNN
-F 2 "" H 4350 6450 60  0001 C CNN
-F 3 "" H 4350 6450 60  0001 C CNN
-	1    4350 6450
-	1    0    0    -1
-$EndComp
-Wire Wire Line
-	5200 5850 4350 5850
-Wire Wire Line
-	4350 5850 4350 5950
-Wire Wire Line
-	4350 6350 4350 6450
-Text Label 2700 8900 2    60   ~ 0
-P2.2/A2
 Text Label 2700 9650 2    60   ~ 0
-P2.1/A1
+P2.5/A5
 NoConn ~ 3850 9550
 Text Notes 7600 8100 0    60   ~ 0
 CL=((C1 x C2) / (C1 + C2)) + 2.5p
+Wire Wire Line
+	5200 5850 4750 5850
+Text Label 2700 8900 2    60   ~ 0
+P3.6
 $EndSCHEMATC
