File: kicad/panstick/panstick.sch (KiCad schematic (older format))
At the start: 25 parts, among them J1 USB_2, P1 CONN_10, P2 CONN_10, SW1 SW_PUSH_SMALL, U1 PANSTAMP_NRG, U2 FT232RL, U3 MCP1702, U4 LY-SK10

Commit message: PCB updated
Connections:
- net D0: now also U4.6
- net D4: now also U4.4; no longer R1.2
- net LED: now reaches U4.5
- net LED: now also R1.2
- no-connect marks 13 -> 10
Other:
- moved on the sheet: D1, R1
Changed lines of the file:
@@
 LIBS:toshiba
 LIBS:panstick-cache
-EELAYER 24 0
+EELAYER 25 0
 EELAYER END
 $Descr A4 11693 8268
@@
 L R R1
 U 1 1 532507A1
-P 4350 2800
-F 0 "R1" V 4430 2800 50  0000 C CNN
-F 1 "1k" V 4350 2800 50  0000 C CNN
-F 2 "SM0603S" H 4350 2800 60  0001 C CNN
-F 3 "" H 4350 2800 60  0001 C CNN
-	1    4350 2800
+P 4750 3650
+F 0 "R1" V 4830 3650 50  0000 C CNN
+F 1 "1k" V 4750 3650 50  0000 C CNN
+F 2 "SM0603S" H 4750 3650 60  0001 C CNN
+F 3 "" H 4750 3650 60  0001 C CNN
+	1    4750 3650
 	0    1    1    0
 $EndComp
 Wire Wire Line
-	3800 2800 4100 2800
+	3800 2800 4150 2800
 $Comp
 L LED D1
 U 1 1 53250A4D
-P 4750 3100
-F 0 "D1" H 4750 3200 50  0000 C CNN
-F 1 "LED" H 4750 3000 50  0000 C CNN
-F 2 "SM0603S_POL" H 4750 3100 60  0001 C CNN
-F 3 "" H 4750 3100 60  0000 C CNN
-	1    4750 3100
+P 5150 3950
+F 0 "D1" H 5150 4050 50  0000 C CNN
+F 1 "LED" H 5150 3850 50  0000 C CNN
+F 2 "SM0603S_POL" H 5150 3950 60  0001 C CNN
+F 3 "" H 5150 3950 60  0000 C CNN
+	1    5150 3950
 	0    1    1    0
 $EndComp
@@
 L GND #PWR021
 U 1 1 53250B0D
-P 4750 3350
-F 0 "#PWR021" H 4750 3350 30  0001 C CNN
-F 1 "GND" H 4750 3280 30  0001 C CNN
-F 2 "" H 4750 3350 60  0001 C CNN
-F 3 "" H 4750 3350 60  0001 C CNN
-	1    4750 3350
-	1    0    0    -1
-$EndComp
-Wire Wire Line
-	4600 2800 4750 2800
-Wire Wire Line
-	4750 2800 4750 2900
+P 5150 4200
+F 0 "#PWR021" H 5150 4200 30  0001 C CNN
+F 1 "GND" H 5150 4130 30  0001 C CNN
+F 2 "" H 5150 4200 60  0001 C CNN
+F 3 "" H 5150 4200 60  0001 C CNN
+	1    5150 4200
+	1    0    0    -1
+$EndComp
+Wire Wire Line
+	5000 3650 5150 3650
+Wire Wire Line
+	5150 3650 5150 3750
 Text Label 4150 2900 2    60   ~ 0
 D5
 Text Label 4150 2700 2    60   ~ 0
 D3
-Text Label 3950 2800 0    60   ~ 0
+Text Label 4150 2800 2    60   ~ 0
 D4
 Text Label 4150 2600 2    60   ~ 0
@@
 D0
 Wire Wire Line
-	4750 3300 4750 3350
+	5150 4150 5150 4200
 Wire Wire Line
 	3050 4800 3500 4800
@@
 	0    -1   -1   0
 $EndComp
-NoConn ~ 4150 950
-NoConn ~ 4250 950
-NoConn ~ 4350 950
 Wire Wire Line
 	3800 2200 4150 2200
 Text Label 4150 2200 2    60   ~ 0
 TEST
+Wire Wire Line
+	4500 3650 4200 3650
+Text Label 4200 3650 0    60   ~ 0
+LED
+Wire Wire Line
+	4250 950  4250 750
+Wire Wire Line
+	4250 750  4600 750
+Text Label 4600 750  2    60   ~ 0
+LED
+Wire Wire Line
+	4350 950  4350 900
+Wire Wire Line
+	4350 900  4600 900
+Text Label 4600 900  2    60   ~ 0
+D4
+Wire Wire Line
+	4150 950  4150 900
+Wire Wire Line
+	4150 900  3900 900
+Text Label 3900 900  0    60   ~ 0
+D0
 $EndSCHEMATC
