File: kicad/addr-rgb-driver/addr-rgb-driver.kicad_pcb (KiCad board)
At the start: 2 copper layers, 21 parts, among them P1 CONN_01X02, P2 CONN_01X03, P3 CONN_01X03, P4 CONN_01X03, P5 CONN_01X03, SW1 SW_PUSH_SMALL, U1 PANSTAMP_NRG, U2 M74VHC1GT08, U3 M74VHC1GT08, U4 M74VHC1GT08, U5 MCP1702, U6 M74VHC1GT08

Commit message: board updated
Parts:
- added G***: PANSTAMPLOGO, PANSTAMPLOGO, F.Cu at (157.2, 100.6)
- C1: footprint old_mysmd:SMDCPOL_10 -> SMDCPOL_10
- C10, C7, C8, C9, R1, R2, R3, R4: footprint old_mysmd:SM0603S -> SM0603S
- P1: footprint old_myconnectors:terminal_block_5mm_2P -> terminal_block_5mm_2P
- P2, P3, P4, P5: footprint old_myconnectors:terminal_block_5mm_3P -> terminal_block_5mm_3P
- SW1: footprint old_mysmd:switch-tact-noah -> switch-tact-noah
- U1: footprint old_mymods:PANSTAMP_NRG -> PANSTAMP_NRG
- U2, U3, U4, U6: footprint libcms:SOT23-5 -> SOT23-5
- U5: footprint mysmd:SOT23 -> SOT23
- moved P2 131.7 mm to (179.0, 100.2), turned to 90 degrees
- moved C7 107.3 mm to (164.3, 118.1), turned to 270 degrees
- moved C8 106.1 mm to (166.3, 118.1), turned to 270 degrees
- moved C9 100.2 mm to (165.1, 111.5), turned to 180 degrees
- moved R1 98.0 mm to (171.9, 88.1), turned to 180 degrees
- moved C10 96.6 mm to (165.1, 109.6), turned to 180 degrees
- moved P5 96.1 mm to (179.0, 85.2)
- moved U1 93.7 mm to (159.9, 92.9)
- moved SW1 93.3 mm to (173.3, 113.9), turned to 270 degrees
- moved U4 91.3 mm to (171.9, 85.0), turned to 270 degrees
- moved R4 90.9 mm to (171.9, 100.5), turned to 180 degrees
- moved P3 88.5 mm to (140.8, 85.1)
- moved U5 78.2 mm to (165.1, 114.3), turned to 90 degrees
- moved U6 78.2 mm to (171.9, 97.4), turned to 270 degrees
- moved U2 67.5 mm to (147.9, 100.1), turned to 90 degrees
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Routing:
- net +5V: track 0.00 -> 157.7 mm
- net /D18: track 0.00 -> 28.5 mm
- net GND: track 0.00 -> 22.6 mm, vias 0 -> 8
- net /D17: track 0.00 -> 20.2 mm
- net /D14: track 0.00 -> 12.0 mm
- net +3.3V: track 0.00 -> 10.4 mm
- net /DATA0: track 0.00 -> 8.70 mm
- net Net-(SW1-Pad2): track 0.00 -> 8.14 mm
- net /DATA3: track 0.00 -> 7.51 mm
- net /DATA2: track 0.00 -> 6.47 mm
- net /DATA1: track 0.00 -> 6.33 mm
- net /D15: track 0.00 -> 4.13 mm
- net Net-(R3-Pad2): track 0.00 -> 4.01 mm
- net Net-(R1-Pad2): track 0.00 -> 3.74 mm
- net Net-(R4-Pad2): track 0.00 -> 3.46 mm
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- added copper zone on F.Cu, net +5V
- added copper zone on B.Cu, net GND
- added copper zone on F.Cu, net GND
Other:
- board outline added: 51.8 x 43.8 mm
- net class Default: clearance 0.2032 -> 0.254; via_dia 1.016 -> 0.889; via_drill 0.6096 -> 0.635
- rule pad_to_mask_clearance: 0 -> 0.2
- rule trace_clearance: 0.2032 -> 0.254
- rule trace_min: 0.2032 -> 0.254
- rule via_min_drill: 0.6096 -> 0.508
- rule via_min_size: 1.016 -> 0.889
- board text added: "+5V GND"
- board text added: "Addressable RGB driver v.1.0"
- board text added: "GND DO0 +5V"
- board text added: "GND DO1 +5V"
- board text added: "GND DO2 +5V"
- board text added: "GND DO3 +5V"
- board text added: "RESET"
- board text added: "www.panstamp.com"
