File: kicad/dipadapter-avr/dipadapter-avr.kicad_pcb (KiCad board)
At the start: 4 copper layers, 3 parts, among them U1 ANTENNA, U2 PANSTAMP_02

Commit message: DIP adapter layout
Parts:
- moved PS1 37.4 mm to (148.4, 91.8)
Other:
- board outline added: 22.2 x 32.8 mm

Commit message: Layout finished
Parts:
- added G***: PANSTAMPLOGO, mymods:PANSTAMPLOGO, F.Cu at (145.7, 99.1)
Routing:
- net GND: track 0.00 -> 95.9 mm, vias 0 -> 11
- net /A0: track 0.00 -> 23.5 mm, vias 0 -> 1
- net /SPI_MOSI: track 0.00 -> 22.4 mm, vias 0 -> 1
- net /A4: track 0.00 -> 21.7 mm, vias 0 -> 1
- net /SPI_SCK: track 0.00 -> 20.6 mm, vias 0 -> 1
- net /A5: track 0.00 -> 18.7 mm, vias 0 -> 1
- net /SPI_MISO: track 0.00 -> 17.5 mm, vias 0 -> 1
- net VCC: track 0.00 -> 16.8 mm, vias 0 -> 2
- net /PD7: track 0.00 -> 16.2 mm, vias 0 -> 1
- net /RESET: track 0.00 -> 15.9 mm, vias 0 -> 1
- net /A7: track 0.00 -> 15.7 mm, vias 0 -> 1
- net /A1: track 0.00 -> 14.9 mm, vias 0 -> 1
- net /A6: track 0.00 -> 14.6 mm, vias 0 -> 1
- net /PD1: track 0.00 -> 14.1 mm, vias 0 -> 1
- net /PB0: track 0.00 -> 12.0 mm, vias 0 -> 1
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- added copper zone on B.Cu, net GND
- added copper zone on F.Cu, net GND
Other:
- board text added: "DIP adapter brd for AVR"
